File: 1590B/1590B.kicad_pcb (KiCad board)
At the start: 2 copper layers, 55.5 x 100 mm, 16 parts, among them J1 V+ GND, J2 IN, J3 OUT, J4 V+ GND, SW1 SW_3PDT

Commit message: WIP
Parts:
- C1: value 0.1 -> 100nF
- C2: value 100 -> 100uF
- J1, J4: footprint Pin_Headers:Pin_Header_Straight_1x02_Pitch2.54mm -> Connector_PinHeader_2.54mm:PinHeader_1x02_P2.54mm_Vertical
- J2: value IN -> NMJ6HCD2; footprint Connectors:NMJ6HCD2 -> Connector_Audio:Jack_6.35mm_Neutrik_NMJ6HCD2_Horizontal
- J3: value OUT -> NMJ6HCD2; footprint Connectors:NMJ6HCD2 -> Connector_Audio:Jack_6.35mm_Neutrik_NMJ6HCD2_Horizontal
- SW1: footprint KiCad Lib:3PDT-Footswitch -> Pedal-Components:3PDT-Footswitch
- moved J3 12.8 mm to (135.0, 130.7), turned to 180 degrees
- moved J2 12.7 mm to (150.6, 114.5), turned to 0 degrees
Connections:
- SW1 pad 4: Net-(J1-T) -> Net-(SW1A-B)
- SW1 pad 5: Net-(J4-T) -> Net-(SW1B-B)
Routing:
- net Net-(SW1A-B): track 0.00 -> 33.5 mm
- net Net-(J2-T): track 33.5 -> 0.00 mm
- net Net-(SW1B-B): track 0.00 -> 21.2 mm
- net Net-(J3-T): track 21.2 -> 0.00 mm
