File: 1590B/untitled.kicad_sch (KiCad schematic)
At the start: 14 parts, among them J1 V+ GND, J2 IN, J3 OUT, J4 V+ GND, SW1 SW_3PDT

Commit message: WIP
Parts:
- removed J2: IN, Connector_Audio:Jack_6.35mm_Neutrik_NMJ6HCD2_Horizontal, symbol 1590B-rescue:JACK_TRS_6PINS-conn
- removed J3: OUT, Connector_Audio:Jack_6.35mm_Neutrik_NMJ6HCD2_Horizontal, symbol 1590B-rescue:JACK_TRS_6PINS-conn
- added J2, J3: NMJ6HCD2, Connector_Audio:Jack_6.35mm_Neutrik_NMJ6HCD2_Horizontal, symbol Connector_Audio:NMJ6HCD2
- SW1: footprint KiCad Lib:3PDT-Footswitch -> Pedal-Components:3PDT-Footswitch
Connections:
- net GND: now also J2.S, J2.TN, J3.S
- net at SW1.5 (B): now also J3.T
- net at SW1.4 (B): now also J2.T
