File: Rebote2.5/Rebote2.5.kicad_pcb (KiCad board)
At the start: 2 copper layers, 55.5 x 100 mm, 63 parts, among them J1 V+ GND, J2 IN, J3 OUT, SW1 SW_3PDT, U1 TL072, U2 L78L05_TO92, U3 PT2399

Commit message: WIP
Parts:
- removed J3: OUT, Connectors:NMJ6HCD2
- C12, C13, C14, C15, C17, C18, C19, C2, C20, C25, C26, C4, C5, C6, C7, C9: footprint Capacitor_THT:C_Rect_L7.0mm_W3.5mm_P2.50mm_P5.00mm -> Capacitor_SMD:C_0805_2012Metric_Pad1.18x1.45mm_HandSolder
- J1: value V+ GND -> NMJ6HCD2; footprint Pin_Headers:Pin_Header_Straight_1x02_Pitch2.54mm -> Connector_Audio:Jack_6.35mm_Neutrik_NMJ6HCD2_Horizontal
- J4: renamed from J2; value IN -> NMJ6HCD2; footprint Connectors:NMJ6HCD2 -> Connector_Audio:Jack_6.35mm_Neutrik_NMJ6HCD2_Horizontal
- R1, R10, R11, R12, R13, R14, R15, R16, R17, R18, R19, R2, R20, R21, R3, R4, R5, R6, R7, R8, R9: footprint Resistor_THT:R_Axial_DIN0207_L6.3mm_D2.5mm_P7.62mm_Horizontal -> Resistor_SMD:R_0805_2012Metric_Pad1.20x1.40mm_HandSolder
- U1: footprint Package_DIP:DIP-8_W7.62mm -> Package_SO:SOIC-8_3.9x4.9mm_P1.27mm
- U2: value L78L05_TO92 -> L78L05_SOT89; footprint Package_TO_SOT_THT:TO-92_Inline -> Package_TO_SOT_SMD:SOT-89-3
- U3: footprint Package_DIP:DIP-16_W7.62mm -> Package_SO:SOIC-16_3.9x9.9mm_P1.27mm
- moved J1 78.2 mm to (135.0, 130.8), turned to 180 degrees
- moved J4 12.7 mm to (150.5, 114.5), turned to 0 degrees
Connections:
- R23 pad 1: O -> Net-(D1-K)
- R23 pad 2: GND -> Net-(SW1C-C)
- R24 pad 1: Net-(D1-K) -> O
- R24 pad 2: Net-(SW1C-C) -> GND
- SW1 pad 4: Net-(J1-T) -> Net-(SW1A-B)
- SW1 pad 5: Net-(J4-T) -> Net-(SW1B-B)
Routing:
- net +9V: track 163.8 -> 0.00 mm
- net I: track 60.7 -> 0.00 mm
- net O: track 53.9 -> 0.00 mm
- net Net-(R12-Pad2): track 52.2 -> 0.00 mm
- net Net-(C6-Pad2): track 47.0 -> 0.00 mm
- net Net-(C21-Pad2): track 36.8 -> 0.00 mm
- net VD: track 30.7 -> 0.00 mm
- net Net-(R15-Pad2): track 27.0 -> 0.00 mm
- net AI: track 26.3 -> 0.00 mm
- net DELAY_OUT: track 24.3 -> 0.00 mm
- net Net-(U1A--): track 22.7 -> 0.00 mm
- net Net-(U3-VCO): track 22.1 -> 0.00 mm
- net Net-(C22-Pad2): track 21.9 -> 0.00 mm
- net LPF2-OUT: track 21.4 -> 0.00 mm
- net +5V: track 20.2 -> 0.00 mm
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